File: bldc_servo_50a_v1.kicad_sch (KiCad schematic)
At the start: 105 parts, among them IC1 DRV8305NQPHPRQ1, J1 CAN_JST-1, J2 CAN_JST-2, J3 Fan_JST, J4 PVDD, J5 GND, J6 SWD, Q1 BSC010N04LS, Q2 BSC010N04LS, Q3 BSC010N04LS, Q4 BSC010N04LS, Q5 BSC010N04LS, Q6 BSC010N04LS, U1 TLV75533PDBV, U2 SN65HVD230, U3 LMR51430, U4 TPS2051BDBV, U5 STM32G431CBT6

Commit message: Update TODO, schematic improvements.
Parts:
- removed A1: A, Solder_Pads:Solder_Pad_5mmx4mm, symbol Connector:Conn_01x01_Pin
- removed B1: B, Solder_Pads:Solder_Pad_5mmx4mm, symbol Connector:Conn_01x01_Pin
- removed C28: C, Solder_Pads:Solder_Pad_5mmx4mm, symbol Connector:Conn_01x01_Pin
- removed D2, D3: SMAJ440A_TVS, Diode_SMD:D_SMA-SMB_Universal_Handsoldering, symbol Diode:SMAJ440A
- removed D7: WS2812, LED_SMD:LED_WS2812_PLCC6_5.0x5.0mm_P1.6mm, symbol LED:WS2812
- removed GH1: 10k, Resistor_SMD:R_0402_1005Metric_Pad0.72x0.64mm_HandSolder, symbol Device:R_Small
- removed J1: CAN_JST-1, Connector_JST:JST_EH_B3B-EH-A_1x03_P2.50mm_Vertical, symbol Connector:Conn_01x03_Pin
- removed J2: CAN_JST-2, Connector_JST:JST_EH_B3B-EH-A_1x03_P2.50mm_Vertical, symbol Connector:Conn_01x03_Pin
- removed J3: Fan_JST, Connector_JST:JST_EH_B3B-EH-A_1x03_P2.50mm_Vertical, symbol Connector:Conn_01x03_Pin
- removed J4: PVDD, Solder_Pads:Solder_Pad_5mmx4mm, symbol Connector:Conn_01x01_Pin
- removed J5: GND, Solder_Pads:Solder_Pad_5mmx4mm, symbol Connector:Conn_01x01_Pin
- removed J6: SWD, Connector_PinHeader_2.54mm:PinHeader_1x05_P2.54mm_Vertical, symbol Connector:Conn_01x05_Pin
- removed U4: TPS2051BDBV, Package_TO_SOT_SMD:SOT-23-5, symbol Power_Management:TPS2051CDBV
- added C28, C50: 4.7u, Capacitor_SMD:C_1206_3216Metric_Pad1.33x1.80mm_HandSolder, symbol Device:C_Small
- added C43: 100n, Capacitor_SMD:C_0402_1005Metric_Pad0.74x0.62mm_HandSolder, symbol Device:C_Small
- added C44, C45, C46, C47, C48, C49: 100u, Capacitor_SMD:CP_Elec_10x7.9, symbol Device:C_Polarized_Small
- added D2: WS2812B-2020, LED_SMD:LED_WS2812B-2020_PLCC4_2.0x2.0mm, symbol LED:WS2812B-2020
- added D3: SMBJ28A, Diode_SMD:D_SMB_Handsoldering, symbol Device:D_Zener_Small
- added H1, H2, H3: ~, positive_altitude:Positive_Altitude_M2_Hole, symbol Mechanical:MountingHole_Pad
- added IC2: TPS22919DCKR, SOT65P210X110-6N, symbol TPS22919DCKR:TPS22919DCKR
- added J2: CAN2, symbol Connector_Generic_MountingPin:Conn_01x03_MountingPin
- added J3: Motor, symbol Connector_Generic:Conn_01x03
- added J4: SWD, positive_altitude:Positive_Altitude_SWD_Connector, symbol positive_altitude:Positive_Altitude_SWD_Connector
- added J5: FAN, symbol Connector_Generic_MountingPin:Conn_01x03_MountingPin
- added J8: Input, symbol Connector_Generic:Conn_01x02
- added TH1: NCP15XH103F03RC, Resistor_SMD:R_0402_1005Metric_Pad0.72x0.64mm_HandSolder, symbol Device:Thermistor_NTC
- C1, C17, C2, C3, C30, C38, C40, C41, C9: footprint Capacitor_SMD:C_0402_1005Metric_Pad0.74x0.62mm_HandSolder -> Capacitor_SMD:C_0603_1608Metric_Pad1.08x0.95mm_HandSolder; LCSC  C106254 -> (none)
- C10, C11: value 470u -> 4.7u; footprint Capacitor_THT:C_Radial_D10.0mm_H16.0mm_P5.00mm -> Capacitor_SMD:C_1206_3216Metric_Pad1.33x1.80mm_HandSolder; LCSC  C51953324 -> C77096
- C12, C16, C8: footprint Capacitor_SMD:C_0402_1005Metric_Pad0.74x0.62mm_HandSolder -> Capacitor_SMD:C_0603_1608Metric_Pad1.08x0.95mm_HandSolder
- C13: value 0.1u -> 4.7u; footprint Capacitor_SMD:C_0402_1005Metric_Pad0.74x0.62mm_HandSolder -> Capacitor_SMD:C_1206_3216Metric_Pad1.33x1.80mm_HandSolder; LCSC  C77020 -> C77096
- C14: value 0.01u -> 4.7u; footprint Capacitor_SMD:C_0402_1005Metric_Pad0.74x0.62mm_HandSolder -> Capacitor_SMD:C_1206_3216Metric_Pad1.33x1.80mm_HandSolder; LCSC  C77019 -> C77096
- C15, C27, C4: value 1u -> 4.7u; footprint Capacitor_SMD:C_0603_1608Metric_Pad1.08x0.95mm_HandSolder -> Capacitor_SMD:C_1206_3216Metric_Pad1.33x1.80mm_HandSolder; LCSC  C559769 -> C77096
- C18, C20, C21, C22, C23, C32, C39, C42: LCSC  C77020 -> (none)
- C19: value 10u -> 4.7u; footprint Capacitor_SMD:C_0805_2012Metric_Pad1.18x1.45mm_HandSolder -> Capacitor_SMD:C_0603_1608Metric_Pad1.08x0.95mm_HandSolder; LCSC  C84416 -> (none)
- C24, C25, C26: LCSC  C77023 -> (none)
- C29: LCSC  C77019 -> (none)
- C34: value 10u -> 4.7u; footprint Capacitor_SMD:C_0805_2012Metric_Pad1.18x1.45mm_HandSolder -> Capacitor_SMD:C_1206_3216Metric_Pad1.33x1.80mm_HandSolder; LCSC  (none) -> C77096
- C5, C6: value 0.047u -> 47n; LCSC  C106260 -> (none)
- C7: footprint Capacitor_SMD:C_0402_1005Metric_Pad0.74x0.62mm_HandSolder -> Capacitor_SMD:C_1206_3216Metric_Pad1.33x1.80mm_HandSolder; LCSC  C132170 -> C77096
- D1: LCSC  couldnt find any -> (none)
- FB1: LCSC  hi -> (none)
- FPC1: value External sensor -> Encoder1
- FPC2: value External sensor -> Encoder2
- L1: footprint Capacitor_SMD:C_0402_1005Metric_Pad0.74x0.62mm_HandSolder -> Inductor_SMD:L_Changjiang_FXL0420
- R1, R12, R13, R15, R16, R17, R2, R7, R8: value 10 -> 10?; LCSC  C109318 -> (none)
- R22, R25, R27: LCSC  C477765 -> (none)
- R23: value 10k1 -> 10k; LCSC  C60490 -> (none)
- R3, R4: LCSC  C60490 -> (none)
Connections:
- net +24V: now also C10.2, C11.2, C13.2, C14.2, C15.2, C27.2, C4.2, C28.1, C44.1, C45.1, C46.1, C47.1, C48.1, C49.1, C50.2, D3.1 (K), J8.1 (Pin_1); no longer C10.1, C11.1, C13.1, C14.1, C15.1, C27.1, C4.1
- net +3.3V: now also J4.1 (+3.3V)
- net +5V: now also C43.1, D2.4 (VDD), IC2.1 (IN)
- net CAN_H: now also J2.1 (Pin_1), J5.1 (Pin_1)
- net CAN_L: now also J2.2 (Pin_2), J5.2 (Pin_2)
- net FAN: now also J5.3 (Pin_3)
- net GND: now also C10.1, C11.1, C12.2, C13.1, C14.1, C15.1, C16.2, C27.1, C4.1, R18.2, R5.2, R9.2, U1.2 (GND), C28.2, C43.2, C44.2, C45.2, C46.2, C47.2, C48.2, C49.2, C50.1, D2.2 (VSS), D3.2 (A), H1.1, H2.1, H3.1, IC2.2 (GND), J2.3 (Pin_3), J4.3 (GND), J5.2 (Pin_2), J5.3 (Pin_3), J8.2 (Pin_2), TH1.2; no longer C10.2, C11.2, C13.2, C14.2, C15.2, C27.2, C4.2
- net LED: now also D2.3 (DIN)
- net NRST: now also J4.5 (RESET)
- net PHASE_A: now also J3.1 (Pin_1)
- net PHASE_B: now also J3.2 (Pin_2)
- net PHASE_C: now also J3.3 (Pin_3)
- net SP1: no longer R5.2
- net SP2: no longer R9.2
- net SP3: no longer R18.2
- net SWCLK: now also J4.2 (SWCLK)
- net SWDIO: now also J4.4 (SWDIO)
- net TEMP: now also TH1.1
- net at IC1.48 (VREG): no longer C1.2
- new net FAN_5V: IC2.6 (OUT), J5.1 (Pin_1)
- new net FAN_EN: IC2.3 (ON)
- no-connect marks 13 -> 17
Other:
- note added: "ADD resistor for VREG!"
- note removed: "Can also use bidirectional instead of uni here"
- note removed: "Changed symbol here"
- note removed: "FAN JST"
- note removed: "Power sw"
- note removed: "add 5v regulator-done"
- note removed: "power distribution switch"
- moved on the sheet: C1, C17, C18, C19, C20, C21, C22, C23, C29, C30, C32, D1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

Commit message: Assign all footprints
Parts:
- removed D1: D_Schottky, symbol Device:D_Schottky
- removed J3: Motor, symbol Connector_Generic:Conn_01x03
- removed J8: Input, symbol Connector_Generic:Conn_01x02
- removed R10, R21, R24, R26: 34.8k, Resistor_SMD:R_0402_1005Metric_Pad0.72x0.64mm_HandSolder, symbol Device:R
- removed R11, R22, R25, R27: 5k, Resistor_SMD:R_0402_1005Metric_Pad0.72x0.64mm_HandSolder, symbol Device:R
- added C51, C52, C53: 1u, Capacitor_SMD:C_0603_1608Metric_Pad1.08x0.95mm_HandSolder, symbol Device:C_Small
- added D7: BAT54SW, Package_TO_SOT_SMD:SOT-323_SC-70, symbol Diode:BAT54SW
- added J3: SWD, Connector_PinHeader_2.54mm:PinHeader_1x05_P2.54mm_Vertical, symbol Connector_Generic:Conn_01x05
- added J5: FAN, Connector_JST:JST_PH_S3B-PH-SM4-TB_1x03-1MP_P2.00mm_Horizontal, symbol Connector_Generic_MountingPin:Conn_01x03_MountingPin
- added NT10, NT11, NT12, NT4, NT5, NT6, NT7, NT8, NT9: NetTie_2, positive_altitude:NetTie-2_SMD_Pad0.2mm, symbol Device:NetTie_2
- added P1: PVDD, positive_altitude:Soldering_Pad_8mm_3mm_hole, symbol Mechanical:MountingHole_Pad
- added P2: GND, positive_altitude:Soldering_Pad_8mm_3mm_hole, symbol Mechanical:MountingHole_Pad
- added P3: PHASE_A, positive_altitude:Soldering_Pad_8mm_3mm_hole, symbol Mechanical:MountingHole_Pad
- added P4: PHASE_B, positive_altitude:Soldering_Pad_8mm_3mm_hole, symbol Mechanical:MountingHole_Pad
- added P5: PHASE_C, positive_altitude:Soldering_Pad_8mm_3mm_hole, symbol Mechanical:MountingHole_Pad
- added R28: 220, Resistor_SMD:R_0402_1005Metric_Pad0.72x0.64mm_HandSolder, symbol Device:R
- added R29, R31, R33, R35: 39k, Resistor_SMD:R_0402_1005Metric_Pad0.72x0.64mm_HandSolder, symbol Device:R
- added R30, R32, R34, R36: 5k, Resistor_SMD:R_0402_1005Metric_Pad0.72x0.64mm_HandSolder, symbol Device:R
- C1: value 1u -> 47n; footprint Capacitor_SMD:C_0603_1608Metric_Pad1.08x0.95mm_HandSolder -> Capacitor_SMD:C_0805_2012Metric_Pad1.18x1.45mm_HandSolder; LCSC  (none) -> C161267; Note (none) -> Should be rated x2 PVDD (100V to be safe), low DC-bias requ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; partno C6119811 -> (none)
- C10, C11, C13, C14, C15, C18, C20, C21, C22, C23, C27, C28, C31, C32, C34, C36, C39, C4, C42, C43, C50, C7: Note (none) -> 50V
- C24, C25, C26: value 22n -> 1n; footprint Capacitor_SMD:C_0402_1005Metric_Pad0.74x0.62mm_HandSolder -> Capacitor_SMD:C_0603_1608Metric_Pad1.08x0.95mm_HandSolder; LCSC  (none) -> C77026; Note (none) -> C0G/NP0
- C33, C35: value 10u -> 22u; LCSC  (none) -> C86816
- C37: value 10u -> 1u; footprint Capacitor_SMD:C_0805_2012Metric_Pad1.18x1.45mm_HandSolder -> Capacitor_SMD:C_0603_1608Metric_Pad1.08x0.95mm_HandSolder
- C5: footprint Capacitor_SMD:C_0402_1005Metric_Pad0.74x0.62mm_HandSolder -> Capacitor_SMD:C_0805_2012Metric_Pad1.18x1.45mm_HandSolder; LCSC  (none) -> C161267; Note (none) -> Should be rated x2 PVDD (100V to be safe), low DC-bias requ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
- C6: value 47n -> 1u; footprint Capacitor_SMD:C_0402_1005Metric_Pad0.74x0.62mm_HandSolder -> Capacitor_SMD:C_0603_1608Metric_Pad1.08x0.95mm_HandSolder
- FB1: value FB -> BLM15AG601SN1D; footprint Capacitor_SMD:C_0402_1005Metric_Pad0.74x0.62mm_HandSolder -> Resistor_SMD:R_0402_1005Metric_Pad0.72x0.64mm_HandSolder; LCSC  (none) -> C76884
- J1: renamed from J5; value FAN -> CAN1; footprint (none) -> Connector_JST:JST_PH_S3B-PH-SM4-TB_1x03-1MP_P2.00mm_Horizontal
- J2: footprint (none) -> Connector_JST:JST_PH_S3B-PH-SM4-TB_1x03-1MP_P2.00mm_Horizontal
- NT1, NT2, NT3: footprint NetTie:NetTie-2_SMD_Pad0.5mm -> positive_altitude:NetTie-2_SMD_Pad0.2mm
- R1, R12, R13, R2, R7, R8: value 10? -> 2.2
- R15, R16, R17: value 10? -> 10
Connections:
- net SH_A_SENSE is gone; now on net PHASE_A_SENSE: U5.11 (PA3)
- net SH_B_SENSE is gone; now on net PHASE_B_SENSE: U5.5 (PF0)
- net SH_C_SENSE is gone; now on net PHASE_C_SENSE: U5.17 (PB1)
- net +24V: now also C17.1, C38.1, C40.1, C41.1, C51.1, C52.1, P1.1, R35.1
- net +3.3V: now also D4.2 (K), D5.2 (K), D6.2 (K), D7.2 (K), J3.1 (Pin_1), R28.1; no longer C1.1
- net +3V3: no longer D4.2 (K), D5.2 (K), D6.2 (K)
- net +5V: no longer C37.1
- net FAN: now also J5.3 (Pin_3); no longer J1.3 (Pin_3)
- net FAN_5V: now also J5.1 (Pin_1); no longer J1.1 (Pin_1)
- net GND: now also C2.2, C6.2, C51.2, C52.2, C53.2, D7.1 (A), J3.3 (Pin_3), J5.2 (Pin_2), P2.1, R30.2, R32.2, R34.2, R36.2; no longer C2.1, J1.2 (Pin_2)
- net NFAULT: no longer R3.2
- net NRST: now also J3.5 (Pin_5)
- net PHASE_A: now also NT6.2, P3.1, R29.1; no longer IC1.35 (SHA)
- net PHASE_B: now also NT9.2, P4.1, R31.1; no longer IC1.30 (SHB)
- net PHASE_C: now also NT12.2, P5.1, R33.1; no longer IC1.27 (SHC)
- net PWRGD: no longer IC1.13 (PWRGD), R4.2
- net SL_A: now also NT5.1; no longer IC1.23 (SN1), Q2.1 (S_1), Q2.11 (S_4), Q2.2 (S_2), Q2.3 (S_3), R5.1
- net SL_B: now also NT7.1; no longer IC1.21 (SN2), Q4.1 (S_1), Q4.11 (S_4), Q4.2 (S_2), Q4.3 (S_3), R9.1
- net SL_C: now also NT10.1; no longer IC1.19 (SN3), Q6.1 (S_1), Q6.11 (S_4), Q6.2 (S_2), Q6.3 (S_3), R18.1
- net SWCLK: now also J3.2 (Pin_2)
- net SWDIO: now also J3.4 (Pin_4)
- net TEMP: now also C53.1
- net WAKE: no longer IC1.47 (WAKE)
- net DRV_AVDD: now reaches C3.1, IC1.15 (AVDD)
- net DRV_VCP_LSD: now reaches C9.1, IC1.37 (VCP_LSD)
- net DRV_VCPH: now reaches C8.1, IC1.38 (VCPH)
- net DRV_CP2H: now reaches IC1.39 (CP2H)
- net DRV_CP2H: now also C1.1; no longer C6.1
- net DRV_CP2L: now reaches IC1.40 (CP2L)
- net DRV_CP2L: now also C1.2; no longer C6.2
- net DRV_CP1H: now reaches C5.1
- net DRV_CP1H: now also IC1.43 (CP1H); no longer IC1.42 (CP1L)
- net DRV_CP1L: now reaches C5.2
- net DRV_CP1L: now also IC1.42 (CP1L); no longer IC1.43 (CP1H)
- net DRV_VDRAIN: now reaches IC1.44 (VDRAIN), R6.2
- net DRV_DVDD: now reaches IC1.46 (DVDD)
- net DRV_DVDD: now also C2.1; no longer C2.2
- net DRV_VREG: now reaches IC1.48 (VREG)
- net DRV_VREG: now also C6.1, R28.2
- net PHASE_B_SENSE: now reaches D4.3 (COM)
- net PHASE_B_SENSE: now also R31.2, R32.1; no longer C38.1
- net DRV_WAKE: now reaches U5.40 (PB3)
- net DRV_WAKE: now also IC1.47 (WAKE)
- net PHASE_A_SENSE: now reaches D6.3 (COM)
- net PHASE_A_SENSE: now also R29.2, R30.1; no longer C41.1
- net PHASE_C_SENSE: now reaches D5.3 (COM)
- net PHASE_C_SENSE: now also R33.2, R34.1; no longer C40.1
- net NSCS renamed DRV_CS
- net PVDDSENSE renamed PVDD_SENSE
- net PVDD_SENSE: now also C37.1, D7.3 (COM), R35.2, R36.1; no longer C17.1
- net SCK renamed SCLK
- new net: NT4.2, NT5.2, Q2.1 (S_1), Q2.11 (S_4), Q2.2 (S_2), Q2.3 (S_3), R5.1
- new net: NT7.2, NT8.2, Q4.1 (S_1), Q4.11 (S_4), Q4.2 (S_2), Q4.3 (S_3), R9.1
- new net: NT10.2, NT11.2, Q6.1 (S_1), Q6.11 (S_4), Q6.2 (S_2), Q6.3 (S_3), R18.1
- new net DRV_NFAULT: R3.2
- new net DRV_PWRGD: IC1.13 (PWRGD), R4.2
- new net SH_A: IC1.35 (SHA), NT6.1
- new net SH_B: IC1.30 (SHB), NT9.1
- new net SH_C: IC1.27 (SHC), NT12.1
- new net SN1: IC1.23 (SN1), NT4.1
- new net SN2: IC1.21 (SN2), NT8.1
- new net SN3: IC1.19 (SN3), NT11.1
- no-connect marks 17 -> 16
Other:
- note removed: "ADD resistor for VREG!"
- note removed: "Driver side SPI"
- note removed: "Encoder side SPI"
- note removed: "NRST"
- note removed: "short with any GPIO"
- moved on the sheet: C2, C3, C39, C5, C7, C8, C9, D6, H1, H2, H3, IC1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
