File: bldc_servo_50a_v1.kicad_pcb (KiCad board)
At the start: 4 copper layers, 65 x 95 mm, 133 parts, among them J1 CAN1, J2 CAN2, J3 FAN, J5 SWD, P1 PVDD, P2 GND, P3 PHASE_A, P4 PHASE_B, P5 PHASE_C, Q1 BSC010N04LS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

Commit message: Some routing
Parts:
- added H4: ~, MountingHole:MountingHole_2.2mm_M2_Pad, F.Cu at (93.5, 103.8)
- added H5: ~, MountingHole:MountingHole_2.2mm_M2_Pad, F.Cu at (93.5, 94.5)
- moved C47 8.75 mm to (137.2, 37.8)
- moved U6 8.06 mm to (134.8, 37.5)
- moved R12 2.62 mm to (160.8, 50.5), turned to 90 degrees
- moved C46 2.46 mm to (162.5, 50.5)
- moved C44 1.13 mm to (138.1, 41.8), turned to 0 degrees
- moved C45 1.12 mm to (146.1, 41.8)
- moved U4 1.12 mm to (142.5, 41.8)
Connections:
- R28 pad 1: +3V3 -> +3.3V
Routing:
- net /CAN_L: track 0.00 -> 27.5 mm
- net /CAN_H: track 0.00 -> 27.0 mm
- net +3.3V: track 0.00 -> 13.4 mm
- net GND: track 0.00 -> 10.5 mm
- net +5V: track 0.00 -> 9.03 mm
- net /5V_SW: track 0.00 -> 2.88 mm
- net Net-(JP1-A): track 0.00 -> 2.26 mm
- net /TEMP: track 0.00 -> 1.57 mm
- added copper zone on F.Cu, net +3.3V
- added copper zone on F.Cu, net +5V
- added copper zone on F.Cu, net GND
- added copper zone on F.Cu, net PVDD
Other:
- board text added: "FAN PDS"
